Commit message: removed commented code and added README

File: urdf/awl_description.xacro (robot description, xacro)
@@ -46,12 +46,4 @@
   </joint>
   <link name="right_main_wheel">
-    <!-- <visual>
-      <geometry>
-        <cylinder length="${main_wheel_length}" radius="${main_wheel_radius}"/>
-      </geometry>
-      <material name="blue">
-        <color rgba="0 0 0 1"/>
-      </material>
-    </visual> -->
     <visual>
       <geometry>
